File: DragonATXProtoLA.kicad_pcb (KiCad board)
At the start: 2 copper layers, 197 x 66.1 mm, 8 parts, among them J1 TTL1, J2 LV1, J3 LV2, J4 TTL2, J5 TTL3, J6 Chain Front, J7 Chain Rear

Commit message: upgrade card edge spec
Routing:
- net A15: track 24.8 -> 23.4 mm
- net A4: track 24.2 -> 23.4 mm
- net A8: track 24.2 -> 23.4 mm
- net A7: track 24.2 -> 23.4 mm
- net A11: track 24.2 -> 23.4 mm
- net A9: track 24.2 -> 23.4 mm
- net A2: track 24.2 -> 23.4 mm
- net A12: track 26.8 -> 26.0 mm
- net GND: vias 57 -> 67
Other:
- outline, holes or cut-outs redrawn

Commit message: prepare for fabrication
Routing:
- net GND: track 0.00 -> 6.35 mm
Changed lines of the file:
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@@
+	)
+	(segment
+		(start 76.9688 111.6866)
+		(end 76.9688 105.3406)
+		(width 1)
+		(layer "B.Cu")
+		(net 4)
 	)
 	(segment
